File: Bachelor boyz.kicad_sch (KiCad schematic)
At the start: 1 part, among them U1 4001

Commit message: Lagt inn 2 forskjellige mikrokontrollere
Parts:
- removed U1: 4001, symbol 4xxx:4001
- added IC1: STM32U575RGT6TR, QFP50P1200X1200X160-64N, symbol STM32U575RGT6TR:STM32U575RGT6TR
- added IC2: STM32U575VIT6Q, QFP50P1600X1600X160-100N, symbol STM32U575VIT6Q:STM32U575VIT6Q
