File: Bachelor boyz.kicad_pcb (KiCad board)
At the start: 2 copper layers, 0 parts

Commit message: Easter egg test
Routing:
- net (no net): track 813.4 -> 953.8 mm
Changed lines of the file:
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@@
 	)
 	(net 0 "")
+	(gr_circle
+		(center 177 124.5)
+		(end 179.885165 128.5)
+		(stroke
+			(width 0.2)
+			(type default)
+		)
+		(fill no)
+		(layer "F.Cu")
+	)
+	(gr_circle
+		(center 137.5 127)
+		(end 140.5 129)
+		(stroke
+			(width 0.2)
+			(type default)
+		)
+		(fill no)
+		(layer "F.Cu")
+	)
+	(gr_circle
+		(center 177 124.5)
+		(end 176 123)
+		(stroke
+			(width 0.2)
+			(type default)
+		)
+		(fill no)
+		(layer "F.Cu")
+	)
+	(gr_circle
+		(center 137.5 127)
+		(end 138.5 127)
+		(stroke
+			(width 0.2)
+			(type default)
+		)
+		(fill no)
+		(layer "F.Cu")
+	)
+	(segment
+		(start 186 139.5)
+		(end 169.5 139.5)
+		(width 0.2)
+		(layer "F.Cu")
+		(net 0)
+	)
 	(segment
 		(start 103.5 35.5)
@@
 	)
 	(segment
+		(start 153.5 130.5)
+		(end 145.5 138.5)
+		(width 0.2)
+		(layer "F.Cu")
+		(net 0)
+	)
+	(segment
 		(start 85 81)
 		(end 96.5 81)
@@
 	)
 	(segment
+		(start 196.5 113.5)
+		(end 196.5 129)
+		(width 0.2)
+		(layer "F.Cu")
+		(net 0)
+	)
+	(segment
 		(start 102 35)
 		(end 83 35)
@@
 	)
 	(segment
+		(start 153.5 117)
+		(end 153.5 130.5)
+		(width 0.2)
+		(layer "F.Cu")
+		(net 0)
+	)
+	(segment
 		(start 105 35.5)
 		(end 111.5 42)
@@
 	)
 	(segment
+		(start 144 140)
+		(end 132.5 140)
+		(width 0.2)
+		(layer "F.Cu")
+		(net 0)
+	)
+	(segment
 		(start 235.25 36.25)
 		(end 250.25 36.25)
@@
 	)
 	(segment
+		(start 132.5 140)
+		(end 123.5 131)
+		(width 0.2)
+		(layer "F.Cu")
+		(net 0)
+	)
+	(segment
+		(start 123.5 131)
+		(end 123.5 118.5)
+		(width 0.2)
+		(layer "F.Cu")
+		(net 0)
+	)
+	(segment
 		(start 189 38)
 		(end 189.5 38.5)
@@
 	)
 	(segment
+		(start 163 133)
+		(end 159 129)
+		(width 0.2)
+		(layer "F.Cu")
+		(net 0)
+	)
+	(segment
+		(start 196.5 129)
+		(end 186 139.5)
+		(width 0.2)
+		(layer "F.Cu")
+		(net 0)
+	)
+	(segment
 		(start 33 35.5)
 		(end 33 82.5)
@@
 	)
 	(segment
+		(start 145.5 138.5)
+		(end 144 140)
+		(width 0.2)
+		(layer "F.Cu")
+		(net 0)
+	)
+	(segment
 		(start 74.5 55)
 		(end 75 55.5)
@@
 	)
 	(segment
+		(start 169.5 139.5)
+		(end 163 133)
+		(width 0.2)
+		(layer "F.Cu")
+		(net 0)
+	)
+	(segment
 		(start 236.5 85.5)
 		(end 237 86)
@@
 		(width 0.2)
 		(layer "F.Cu")
+		(net 0)
+	)
+	(segment
+		(start 159 129)
+		(end 159 114)
+		(width 0.2)
+		(layer "F.Cu")

Commit message: Fyfaen
Routing:
- net (no net): track 953.8 -> 1223.5 mm
Changed lines of the file:
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@@
+	)
+	(segment
+		(start 43 184.5)
+		(end 35 192.5)
+		(width 0.2)
+		(layer "F.Cu")
+		(net 0)
 	)
 	(segment
@@
 	)
 	(segment
+		(start 25 188.5)
+		(end 16 197.5)
+		(width 0.2)
+		(layer "F.Cu")
+		(net 0)
+	)
+	(segment
 		(start 103.5 35.5)
 		(end 105 35.5)
@@
 	)
 	(segment
+		(start 86 150.5)
+		(end 101 165.5)
+		(width 0.2)
+		(layer "F.Cu")
+		(net 0)
+	)
+	(segment
 		(start 189 38.5)
 		(end 178.5 49)
@@
 	)
 	(segment
+		(start 105 168)
+		(end 86 187)
+		(width 0.2)
+		(layer "F.Cu")
+		(net 0)
+	)
+	(segment
+		(start 40 150)
+		(end 41.5 148.5)
+		(width 0.2)
+		(layer "F.Cu")
+		(net 0)
+	)
+	(segment
 		(start 153.5 130.5)
 		(end 145.5 138.5)
@@
 	)
 	(segment
+		(start 30.5 195)
+		(end 25 189.5)
+		(width 0.2)
+		(layer "F.Cu")
+		(net 0)
+	)
+	(segment
 		(start 224 82)
 		(end 224 51)
@@
 	)
 	(segment
+		(start 83.5 184.5)
+		(end 43 184.5)
+		(width 0.2)
+		(layer "F.Cu")
+		(net 0)
+	)
+	(segment
 		(start 75 71)
 		(end 85 81)
@@
 	)
 	(segment
+		(start 25 185)
+		(end 25 188.5)
+		(width 0.2)
+		(layer "F.Cu")
+		(net 0)
+	)
+	(segment
 		(start 236.5 88.5)
 		(end 236.5 37.5)
@@
 	)
 	(segment
+		(start 16 197.5)
+		(end 14 195.5)
+		(width 0.2)
+		(layer "F.Cu")
+		(net 0)
+	)
+	(segment
 		(start 178.5 49)
 		(end 178.5 81.5)
@@
 	)
 	(segment
+		(start 40 151.5)
+		(end 85 151.5)
+		(width 0.2)
+		(layer "F.Cu")
+		(net 0)
+	)
+	(segment
 		(start 163 133)
 		(end 159 129)
@@
 	)
 	(segment
+		(start 31 195.5)
+		(end 30.5 195)
+		(width 0.2)
+		(layer "F.Cu")
+		(net 0)
+	)
+	(segment
 		(start 249.5 100.5)
 		(end 238 100.5)
@@
 	)
 	(segment
+		(start 85 151.5)
+		(end 86 150.5)
+		(width 0.2)
+		(layer "F.Cu")
+		(net 0)
+	)
+	(segment
 		(start 236.5 85.5)
 		(end 237 86)
@@
 	)
 	(segment
+		(start 105 165.5)
+		(end 105 168)
+		(width 0.2)
+		(layer "F.Cu")
+		(net 0)
+	)
+	(segment
+		(start 13.5 150)
+		(end 40 150)
+		(width 0.2)
+		(layer "F.Cu")
+		(net 0)
+	)
+	(segment
 		(start 61.5 36.5)
 		(end 61.5 80.5)
@@
 	)
 	(segment
+		(start 101 165.5)
+		(end 105 165.5)
+		(width 0.2)
+		(layer "F.Cu")
+		(net 0)
+	)
+	(segment
 		(start 238 100.5)
 		(end 238 92.5)
@@
 	)
 	(segment
+		(start 14 150.5)
+		(end 13.5 150)
+		(width 0.2)
+		(layer "F.Cu")
+		(net 0)
+	)
+	(segment
 		(start 250.5 36.5)
 		(end 250.5 87)
@@
 	)
 	(segment
+		(start 25 189.5)
+		(end 25 185)
+		(width 0.2)
+		(layer "F.Cu")
+		(net 0)
+	)
+	(segment
+		(start 14 166)
+		(end 14 150.5)
+		(width 0.2)
+		(layer "F.Cu")
+		(net 0)
+	)
+	(segment
+		(start 86 187)
+		(end 83.5 184.5)
+		(width 0.2)
+		(layer "F.Cu")
+		(net 0)
+	)
+	(segment
+		(start 35 195.5)
+		(end 31 195.5)
+		(width 0.2)
+		(layer "F.Cu")
+		(net 0)
+	)
+	(segment
+		(start 35 192.5)
+		(end 35 195.5)
+		(width 0.2)
+		(layer "F.Cu")
+		(net 0)
+	)
+	(segment
 		(start 178.5 81.5)
 		(end 188 91)
@@
 		(width 0.2)
 		(layer "F.Cu")
+		(net 0)
+	)
+	(segment
+		(start 14 195.5)
+		(end 14 187.5)
+		(width 0.2)
+		(layer "F.Cu")
+		(net 0)
+	)
+	(segment
+		(start 14 187.5)
+		(end 14 166)
+		(width 0.2)
+		(layer "F.Cu")

Commit message: Lagt inn 2 forskjellige mikrokontrollere
Parts:
- added IC1: STM32U575RGT6TR, STM32U575RGT6TR:QFP50P1200X1200X160-64N, F.Cu at (83.8, 101.8)
- added IC2: STM32U575VIT6Q, STM32U575VIT6Q:QFP50P1600X1600X160-100N, F.Cu at (99.8, 103.8)
